Commit message: Latest Modification

File: turn_on_dlrobot_robot/description/camera.xacro (robot description, xacro)
@@ -4,10 +4,10 @@
         <parent link="chassis"/>
         <child link="camera_link"/>
-        <origin xyz="0.270 0 0.180" rpy="0 0 0"/>
+        <origin xyz="0.580 0 0.430" rpy="0 0 0"/>
     </joint>
     <link name="camera_link">
         <visual>
             <geometry>
-                <box size="0.010 0.06 0.03"/>
+                <box size="0.030 0.15 0.060"/>
             </geometry>
             <material name="red"/>
@@ -16,5 +16,5 @@
             <origin xyz="0 0 -0.05"/>
             <geometry>
-                <cylinder radius="0.002" length="0.1"/>
+                <cylinder radius="0.015" length="0.1"/>
             </geometry>
             <material name="red"/>

File: turn_on_dlrobot_robot/description/lidar.xacro (robot description, xacro)
@@ -4,18 +4,17 @@
         <parent link="chassis"/>
         <child link="laser_frame"/>
-        <origin xyz="0.122 0 0.212" rpy="0 0 0"/>
+        <origin xyz="0.30 0 0.49" rpy="0 0 0"/>
     </joint>
     <link name="laser_frame">
         <visual>
-            <!-- <origin xyz="-0.05 0 0"/> -->
             <geometry>
-                <cylinder radius="0.05" length="0.04"/>
+                <cylinder radius="0.07" length="0.04"/>
             </geometry>
             <material name="red"/>
         </visual>
         <visual>
-            <origin xyz="0 0 -0.05"/>
+            <origin xyz="0 0 -0.09"/>
             <geometry>
-                <cylinder radius="0.01" length="0.1"/>
+                <cylinder radius="0.02" length="0.15"/>
             </geometry>
             <material name="red"/>
@@ -23,8 +22,8 @@
         <collision>
             <geometry>
-                <cylinder radius="0.05" length="0.04"/>
+                <cylinder radius="0.07" length="0.04"/>
             </geometry>
         </collision>
-        <xacro:inertial_cylinder mass="0.1" length="0.04" radius="0.05">
+        <xacro:inertial_cylinder mass="0.1" length="0.04" radius="0.07">
             <origin xyz="0 0 0" rpy="0 0 0"/>
         </xacro:inertial_cylinder>

File: turn_on_dlrobot_robot/description/robot_core.xacro (robot description, xacro)
@@ -2,17 +2,17 @@
 <robot xmlns:xacro="http://www.ros.org/wiki/xacro" >
     <xacro:include filename="inertial_macros.xacro"/>
-    <xacro:property name="chassis_length" value="0.335"/>
-    <xacro:property name="chassis_width" value="0.265"/>
-    <xacro:property name="chassis_height" value="0.138"/>
+    <xacro:property name="chassis_length" value="0.8"/>
+    <xacro:property name="chassis_width" value="0.63"/>
+    <xacro:property name="chassis_height" value="0.33"/>
     <xacro:property name="chassis_mass" value="1.0"/>
-    <xacro:property name="wheel_radius" value="0.034"/>
-    <xacro:property name="wheel_thickness" value="0.026"/>
+    <xacro:property name="wheel_radius" value="0.07"/>
+    <xacro:property name="wheel_thickness" value="0.06"/>
     <xacro:property name="wheel_mass" value="0.05"/>
-    <xacro:property name="wheel_offset_x" value="0.226"/>
-    <xacro:property name="wheel_offset_y" value="0.166"/>
+    <xacro:property name="wheel_offset_x" value="0.60"/>
+    <xacro:property name="wheel_offset_y" value="0.38"/>
     <xacro:property name="wheel_offset_z" value="0.01"/>
-    <xacro:property name="caster_wheel_radius" value="0.01"/>
+    <xacro:property name="caster_wheel_radius" value="0.07"/>
     <xacro:property name="caster_wheel_mass" value="0.01"/>
-    <xacro:property name="caster_wheel_offset_x" value="0.075"/>
+    <xacro:property name="caster_wheel_offset_x" value="0.15"/>
     <xacro:property name="caster_wheel_offset_z" value="${wheel_offset_z - wheel_radius + caster_wheel_radius}"/>
     <material name="white">
